File: HW/current-driver.sch (KiCad schematic (older format))
At the start: 17 parts, among them P1 IN+, P2 IN-, P3 LED, P4 SW_IN, P5 SENSE, P6 OUT+, P7 OUT-, Q1 IRFZ44VBF, U1 INA168

Commit message: Schematic v2b1
Parts:
- added C1: CP, ~, symbol CP
- added D2: BZX55C15, symbol ZENER
- added R7: 6K8 (48V), ~, symbol R
- F1: footprint ~ -> AUTOFUSE
Connections:
- net at P2.1, P4.2 (PM), P5.2 (PM)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: now also C1.2, D2.1 (A)
- net at F1.2, R1.1, R2.2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: now also R7.1; no longer U1.5 (V+)
- new net: C1.1, D2.2 (K), R7.2, U1.5 (V+)
Other:
- moved on the sheet: F1, P1, P2
Changed lines of the file:
@@
 LIBS:contrib
 LIBS:valves
+LIBS:current-driver-cache
 EELAYER 27 0
 EELAYER END
@@
 Sheet 1 1
 Title ""
-Date "23 jul 2014"
+Date "29 jul 2014"
 Rev ""
 Comp ""
@@
 L CONN_1 P1
 U 1 1 53CDE287
-P 2950 2150
-F 0 "P1" H 3030 2150 40  0000 L CNN
-F 1 "IN+" H 2950 2205 30  0000 C CNN
-F 2 "" H 2950 2150 60  0000 C CNN
-F 3 "" H 2950 2150 60  0000 C CNN
-	1    2950 2150
+P 2600 2150
+F 0 "P1" H 2680 2150 40  0000 L CNN
+F 1 "IN+" H 2600 2205 30  0000 C CNN
+F 2 "" H 2600 2150 60  0000 C CNN
+F 3 "" H 2600 2150 60  0000 C CNN
+	1    2600 2150
 	-1   0    0    1
 $EndComp
@@
 L CONN_1 P2
 U 1 1 53CDE2B8
-P 2950 3500
-F 0 "P2" H 3030 3500 40  0000 L CNN
-F 1 "IN-" H 2950 3555 30  0000 C CNN
-F 2 "" H 2950 3500 60  0000 C CNN
-F 3 "" H 2950 3500 60  0000 C CNN
-	1    2950 3500
+P 2600 3500
+F 0 "P2" H 2680 3500 40  0000 L CNN
+F 1 "IN-" H 2600 3555 30  0000 C CNN
+F 2 "" H 2600 3500 60  0000 C CNN
+F 3 "" H 2600 3500 60  0000 C CNN
+	1    2600 3500
 	-1   0    0    1
 $EndComp
 Wire Wire Line
-	5450 3500 3100 3500
+	5450 3500 2750 3500
 $Comp
 L FUSE F1
 U 1 1 53CDE417
-P 3400 2150
-F 0 "F1" H 3500 2200 40  0000 C CNN
-F 1 "FUSE" H 3300 2100 40  0000 C CNN
-F 2 "~" H 3400 2150 60  0000 C CNN
-F 3 "~" H 3400 2150 60  0000 C CNN
-	1    3400 2150
+P 3050 2150
+F 0 "F1" H 3150 2200 40  0000 C CNN
+F 1 "FUSE" H 2950 2100 40  0000 C CNN
+F 2 "AUTOFUSE" H 3050 2150 60  0001 C CNN
+F 3 "~" H 3050 2150 60  0000 C CNN
+	1    3050 2150
 	1    0    0    -1
 $EndComp
@@
 	1    0    0    -1
 $EndComp
-Wire Wire Line
-	4100 2350 4150 2350
-Wire Wire Line
-	4150 2350 4150 2150
-Wire Wire Line
-	3750 2350 3900 2350
-Wire Wire Line
-	3750 1650 3750 2350
-Connection ~ 3800 2350
 $Comp
 L R R4
@@
 Connection ~ 3800 3500
 Wire Wire Line
-	3750 2150 3650 2150
-Wire Wire Line
-	3100 2150 3150 2150
+	3750 2150 3300 2150
+Wire Wire Line
+	2750 2150 2800 2150
 Wire Wire Line
 	4150 2150 5750 2150
@@
 	-1   0    0    -1
 $EndComp
+$Comp
+L R R7
+U 1 1 53D720B3
+P 3350 2400
+F 0 "R7" H 3350 2325 40  0000 C CNN
+F 1 "6K8 (48V)" H 3350 2475 40  0000 C CNN
+F 2 "~" H 3350 2400 60  0000 C CNN
+F 3 "~" H 3350 2400 60  0000 C CNN
+	1    3350 2400
+	0    1    1    0
+$EndComp
+$Comp
+L ZENER D2
+U 1 1 53D720F2
+P 3350 3250
+F 0 "D2" H 3350 3350 50  0000 C CNN
+F 1 "BZX55C15" H 3350 3150 40  0000 C CNN
+F 2 "" H 3350 3250 60  0000 C CNN
+F 3 "" H 3350 3250 60  0000 C CNN
+	1    3350 3250
+	0    -1   -1   0
+$EndComp
+Wire Wire Line
+	3350 3450 3350 3500
+Connection ~ 3350 3500
+Wire Wire Line
+	3350 3050 3350 2600
+Wire Wire Line
+	3350 2200 3350 2150
+Connection ~ 3350 2150
+Wire Wire Line
+	4100 2350 4100 2250
+Wire Wire Line
+	4100 2250 4150 2250
+Wire Wire Line
+	4150 2250 4150 2150
+Wire Wire Line
+	3900 2350 3900 2250
+Wire Wire Line
+	3750 2250 3900 2250
+Wire Wire Line
+	3750 1650 3750 2250
+Wire Wire Line
+	3350 2650 3600 2650
+Wire Wire Line
+	3600 2350 3600 3150
+Wire Wire Line
+	3600 2350 3800 2350
+Connection ~ 3350 2650
+$Comp
+L CP C1
+U 1 1 53D721FC
+P 3600 3250
+F 0 "C1" H 3600 3100 40  0000 C CNN
+F 1 "CP" H 3600 3400 40  0000 C CNN
+F 2 "~" H 3600 3250 60  0000 C CNN
+F 3 "~" H 3600 3250 60  0000 C CNN
+	1    3600 3250
+	0    1    1    0
+$EndComp
+Connection ~ 3600 2650
+Wire Wire Line
+	3600 3350 3600 3500
+Connection ~ 3600 3500
 $EndSCHEMATC

Commit message: Schematic v2 finished netlist/pcb added
Parts:
- C1: value CP -> 10uF/25V; footprint ~ -> C1P_D2
- D1: footprint ~ -> LED3
- D2: footprint (none) -> D3
- P1, P2, P6, P7: footprint (none) -> HEADER_6.3
- P3, P4, P5: footprint (none) -> HDR-2
- R1, R2, R4, R5, R6, R7: footprint ~ -> R4
- R3: footprint ~ -> R4_5_6
- U1: footprint (none) -> SOT23-5
Changed lines of the file:
@@
 Sheet 1 1
 Title ""
-Date "29 jul 2014"
+Date "30 jul 2014"
 Rev ""
 Comp ""
@@
 F 0 "P1" H 2680 2150 40  0000 L CNN
 F 1 "IN+" H 2600 2205 30  0000 C CNN
-F 2 "" H 2600 2150 60  0000 C CNN
+F 2 "HEADER_6.3" H 2600 2150 60  0001 C CNN
 F 3 "" H 2600 2150 60  0000 C CNN
 	1    2600 2150
@@
 F 0 "P6" H 5980 2150 40  0000 L CNN
 F 1 "OUT+" H 5900 2205 30  0000 C CNN
-F 2 "" H 5900 2150 60  0000 C CNN
+F 2 "HEADER_6.3" H 5900 2150 60  0001 C CNN
 F 3 "" H 5900 2150 60  0000 C CNN
 	1    5900 2150
@@
 F 0 "P7" H 5980 2350 40  0000 L CNN
 F 1 "OUT-" H 5900 2405 30  0000 C CNN
-F 2 "" H 5900 2350 60  0000 C CNN
+F 2 "HEADER_6.3" H 5900 2350 60  0001 C CNN
 F 3 "" H 5900 2350 60  0000 C CNN
 	1    5900 2350
@@
 F 0 "P2" H 2680 3500 40  0000 L CNN
 F 1 "IN-" H 2600 3555 30  0000 C CNN
-F 2 "" H 2600 3500 60  0000 C CNN
+F 2 "HEADER_6.3" H 2600 3500 60  0001 C CNN
 F 3 "" H 2600 3500 60  0000 C CNN
 	1    2600 3500
@@
 F 0 "R5" H 5000 2675 40  0000 C CNN
 F 1 "10R" H 5300 2675 40  0000 C CNN
-F 2 "~" H 5150 2600 60  0000 C CNN
+F 2 "R4" H 5150 2600 60  0001 C CNN
 F 3 "~" H 5150 2600 60  0000 C CNN
 	1    5150 2600
@@
 F 0 "R6" H 5025 2675 40  0000 C CNN
 F 1 "100K" H 5300 2675 40  0000 C CNN
-F 2 "~" H 5150 2750 60  0000 C CNN
+F 2 "R4" H 5150 2750 60  0001 C CNN
 F 3 "~" H 5150 2750 60  0000 C CNN
 	1    5150 2750
@@
 F 0 "R3" H 3950 2075 40  0000 C CNN
 F 1 "R005/1W" H 3950 2225 40  0000 C CNN
-F 2 "~" H 3950 2150 60  0000 C CNN
+F 2 "R4_5_6" H 3950 2150 60  0001 C CNN
 F 3 "~" H 3950 2150 60  0000 C CNN
 	1    3950 2150
@@
 F 0 "U1" H 4250 2550 60  0000 C CNN
 F 1 "INA168" H 3550 2900 60  0000 C CNN
-F 2 "" H 4000 2700 60  0000 C CNN
+F 2 "SOT23-5" H 4000 2700 60  0001 C CNN
 F 3 "" H 4000 2700 60  0000 C CNN
 	1    3950 2700
@@
 F 0 "R4" H 4100 3175 40  0000 C CNN
 F 1 "100K" H 4100 3325 40  0000 C CNN
-F 2 "~" H 4100 3250 60  0000 C CNN
+F 2 "R4" H 4100 3250 60  0001 C CNN
 F 3 "~" H 4100 3250 60  0000 C CNN
 	1    4100 3250
@@
 F 0 "R2" H 3950 1825 40  0000 C CNN
 F 1 "10K" H 3950 1975 40  0000 C CNN
-F 2 "~" H 3950 1900 60  0000 C CNN
+F 2 "R4" H 3950 1900 60  0001 C CNN
 F 3 "~" H 3950 1900 60  0000 C CNN
 	1    3950 1900
@@
 F 0 "R1" H 3950 1575 40  0000 C CNN
 F 1 "10K" H 3950 1725 40  0000 C CNN
-F 2 "~" H 3950 1650 60  0000 C CNN
+F 2 "R4" H 3950 1650 60  0001 C CNN
 F 3 "~" H 3950 1650 60  0000 C CNN
 	1    3950 1650
@@
 F 0 "D1" H 4400 2000 50  0000 C CNN
 F 1 "LED" H 4400 1800 50  0000 C CNN
-F 2 "~" H 4400 1900 60  0000 C CNN
+F 2 "LED3" H 4400 1900 60  0001 C CNN
 F 3 "~" H 4400 1900 60  0000 C CNN
 	1    4400 1900
@@
 F 0 "P3" V 5800 1750 40  0000 C CNN
 F 1 "LED" V 5900 1750 40  0000 C CNN
-F 2 "" H 5850 1750 60  0000 C CNN
+F 2 "HDR-2" H 5850 1750 60  0001 C CNN
 F 3 "" H 5850 1750 60  0000 C CNN
 	1    5850 1750
@@
 F 0 "P4" V 5800 2700 40  0000 C CNN
 F 1 "SW_IN" V 5900 2700 40  0000 C CNN
-F 2 "" H 5850 2700 60  0000 C CNN
+F 2 "HDR-2" H 5850 2700 60  0001 C CNN
 F 3 "" H 5850 2700 60  0000 C CNN
 	1    5850 2700
@@
 F 0 "P5" V 5800 3100 40  0000 C CNN
 F 1 "SENSE" V 5900 3100 40  0000 C CNN
-F 2 "" H 5850 3100 60  0000 C CNN
+F 2 "HDR-2" H 5850 3100 60  0001 C CNN
 F 3 "" H 5850 3100 60  0000 C CNN
 	1    5850 3100
@@
 F 0 "R7" H 3350 2325 40  0000 C CNN
 F 1 "6K8 (48V)" H 3350 2475 40  0000 C CNN
-F 2 "~" H 3350 2400 60  0000 C CNN
+F 2 "R4" H 3350 2400 60  0001 C CNN
 F 3 "~" H 3350 2400 60  0000 C CNN
 	1    3350 2400
@@
 F 0 "D2" H 3350 3350 50  0000 C CNN
 F 1 "BZX55C15" H 3350 3150 40  0000 C CNN
-F 2 "" H 3350 3250 60  0000 C CNN
+F 2 "D3" H 3350 3250 60  0001 C CNN
 F 3 "" H 3350 3250 60  0000 C CNN
 	1    3350 3250
@@
 	3900 2350 3900 2250
 Wire Wire Line
-	3750 2250 3900 2250
-Wire Wire Line
-	3750 1650 3750 2250
+	3900 2250 3750 2250
+Wire Wire Line
+	3750 2250 3750 1650
 Wire Wire Line
 	3350 2650 3600 2650
@@
 P 3600 3250
 F 0 "C1" H 3600 3100 40  0000 C CNN
-F 1 "CP" H 3600 3400 40  0000 C CNN
-F 2 "~" H 3600 3250 60  0000 C CNN
+F 1 "10uF/25V" H 3600 3400 40  0000 C CNN
+F 2 "C1P_D2" H 3600 3250 60  0001 C CNN
 F 3 "~" H 3600 3250 60  0000 C CNN
 	1    3600 3250
