File: HW/current-driver.kicad_pcb (KiCad board)
At the start: 2 copper layers, 0 parts

Commit message: Schematic v2 finished netlist/pcb added
Parts:
- added C1: 10uF/25V, C1P_D2, F.Cu at (211.0, 152.0)
- added D1: LED, LED3, F.Cu at (211.0, 152.0)
- added D2: BZX55C15, D3, F.Cu at (211.0, 152.0)
- added F1: FUSE, AUTOFUSE, F.Cu at (162.0, 113.0)
- added P1: IN+, HEADER_6.3, F.Cu at (136.0, 114.0)
- added P2: IN-, HEADER_6.3, F.Cu at (136.0, 127.0)
- added P3: LED, HDR-2, F.Cu at (211.0, 152.0)
- added P4: SW_IN, HDR-2, F.Cu at (211.0, 152.0)
- added P5: SENSE, HDR-2, F.Cu at (211.0, 152.0)
- added P6: OUT+, HEADER_6.3, F.Cu at (211.0, 152.0)
- added P7: OUT-, HEADER_6.3, F.Cu at (211.0, 152.0)
- added Q1: IRFZ44VBF, TO220, F.Cu at (211.0, 152.0)
- added R1, R2: 10K, R4, F.Cu at (211.0, 152.0)
- added R3: R005/1W, R4_5_6, F.Cu at (211.0, 152.0)
- added R4, R6: 100K, R4, F.Cu at (211.0, 152.0)
- added R5: 10R, R4, F.Cu at (211.0, 152.0)
- added R7: 6K8 (48V), R4, F.Cu at (159.0, 127.0)
- added U1: INA168, SOT23-5, F.Cu at (211.0, 152.0)

Commit message: PCB v1b1
Parts:
- U1: moved to B.Cu
- moved D2 99.4 mm to (121.9, 108.0), turned to 90 degrees
- moved C1 93.7 mm to (127.0, 110.5), turned to 270 degrees
- moved P6 93.4 mm to (124.5, 116.8)
- moved R3 91.2 mm to (135.9, 100.3), turned to 270 degrees
- moved P7 90.1 mm to (124.5, 127.0)
- moved R4 83.6 mm to (144.8, 101.0), turned to 180 degrees
- moved R2 81.6 mm to (154.9, 92.7), turned to 90 degrees
- moved U1 80.8 mm to (144.1, 106.7)
- moved R1 79.9 mm to (157.5, 92.7), turned to 270 degrees
- moved Q1 77.6 mm to (143.5, 113.7), turned to 270 degrees
- moved D1 77.2 mm to (153.0, 101.0), turned to 270 degrees
- moved P3 71.3 mm to (158.8, 103.5), turned to 270 degrees
- moved R5 69.0 mm to (150.5, 118.7), turned to 270 degrees
- moved P5 67.9 mm to (158.8, 108.6), turned to 270 degrees
- moved R6 66.8 mm to (153.0, 118.7), turned to 270 degrees
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Routing:
- net N-000006: track 0.00 -> 196.2 mm
- net N-000007: track 0.00 -> 64.4 mm
- net N-0000011: track 0.00 -> 59.1 mm
- net N-000003: track 0.00 -> 38.2 mm, vias 0 -> 2
- net N-000008: track 0.00 -> 32.1 mm
- net N-000004: track 0.00 -> 32.0 mm
- net N-0000010: track 0.00 -> 23.2 mm
- net N-000002: track 0.00 -> 17.1 mm
- net N-000005: track 0.00 -> 4.97 mm
- net N-000001: track 0.00 -> 4.44 mm
- net N-000009: track 0.00 -> 2.69 mm
