File: HW/current-driver_panelize.kicad_pcb (KiCad board)
At the start: 2 copper layers, 268 x 182 mm, 288 parts, among them P1 IN+, P2 IN-, P3 LED, P4 SW_IN, P5 SENSE, P6 OUT+, P7 OUT-, Q1 IRFZ44VBF, U1 INA168

Commit message: Panelized PCB for printing added
Parts:
- removed the C1 at (187.0, 171.5)
- removed the C1 at (88.0, 101.5)
- removed the C1 at (88.0, 44.5)
- removed the C1 at (244.0, 171.5)
- removed the C1 at (88.0, 171.5)
- removed the C1 at (31.0, 171.5)
- removed the C1 at (187.0, 44.5)
- removed the C1 at (244.0, 44.5)
- removed the C1 at (244.0, 101.5)
- removed the C1 at (187.0, 101.5)
- removed the C1 at (31.0, 101.5)
- removed the D1 at (213.0, 170.9)
- removed the D1 at (114.0, 100.9)
- removed the D1 at (114.0, 43.9)
- removed the D1 at (270.0, 170.9)
- removed the D1 at (114.0, 170.9)
- removed the D1 at (57.0, 170.9)
- removed the D1 at (213.0, 43.9)
- removed the D1 at (270.0, 43.9)
- removed the D1 at (270.0, 100.9)
- removed the D1 at (213.0, 100.9)
- removed the D1 at (57.0, 100.9)
- removed the D2 at (181.9, 168.9)
- removed the D2 at (82.9, 99.0)
- removed the D2 at (82.9, 42.0)
- removed the D2 at (238.9, 168.9)
- removed the D2 at (82.9, 168.9)
- removed the D2 at (25.9, 168.9)
- removed the D2 at (181.9, 42.0)
- removed the D2 at (238.9, 42.0)
- removed the D2 at (238.9, 99.0)
- removed the D2 at (181.9, 99.0)
- removed the D2 at (25.9, 99.0)
- removed the F1 at (202.2, 149.9)
- removed the F1 at (103.2, 79.9)
- removed the F1 at (103.2, 22.9)
- removed the F1 at (259.2, 149.9)
- removed the F1 at (103.2, 149.9)
- removed the F1 at (46.2, 149.9)
- removed the F1 at (202.2, 22.9)
- removed the F1 at (259.2, 22.9)
- removed the F1 at (259.2, 79.9)
- removed the F1 at (202.2, 79.9)
- removed the F1 at (46.2, 79.9)
- removed MNT_HOLE_3.5 (x48): , MNT_HOLE_3.5
- removed the P1 at (184.5, 149.9)
- removed the P1 at (85.5, 79.9)
- removed the P1 at (85.5, 22.9)
- removed the P1 at (241.5, 149.9)
- removed the P1 at (85.5, 149.9)
- removed the P1 at (28.5, 149.9)
- removed the P1 at (184.5, 22.9)
- removed the P1 at (241.5, 22.9)
- removed the P1 at (241.5, 79.9)
- removed the P1 at (184.5, 79.9)
- removed the P1 at (28.5, 79.9)
- removed the P2 at (184.5, 160.1)
- removed the P2 at (85.5, 90.1)
- removed the P2 at (85.5, 33.1)
- removed the P2 at (241.5, 160.1)
- removed the P2 at (85.5, 160.1)
- removed the P2 at (28.5, 160.1)
- removed the P2 at (184.5, 33.1)
- removed the P2 at (241.5, 33.1)
- removed the P2 at (241.5, 90.1)
- removed the P2 at (184.5, 90.1)
- removed the P2 at (28.5, 90.1)
- removed the P3 at (218.8, 172.8)
- removed the P3 at (119.8, 102.8)
- removed the P3 at (119.8, 45.8)
- removed the P3 at (275.8, 172.8)
- removed the P3 at (119.8, 172.8)
- removed the P3 at (62.8, 172.8)
- removed the P3 at (218.8, 45.8)
- removed the P3 at (275.8, 45.8)
- removed the P3 at (275.8, 102.8)
- removed the P3 at (218.8, 102.8)
- removed the P3 at (62.8, 102.8)
- removed the P4 at (218.8, 182.9)
- removed the P4 at (119.8, 112.9)
- removed the P4 at (119.8, 55.9)
- removed the P4 at (275.8, 182.9)
- removed the P4 at (119.8, 182.9)
- removed the P4 at (62.8, 182.9)
- removed the P4 at (218.8, 55.9)
- removed the P4 at (275.8, 55.9)
- removed the P4 at (275.8, 112.9)
- removed the P4 at (218.8, 112.9)
- removed the P4 at (62.8, 112.9)
- removed the P5 at (218.8, 177.8)
- removed the P5 at (119.8, 107.8)
- removed the P5 at (119.8, 50.8)
- removed the P5 at (275.8, 177.8)
- removed the P5 at (119.8, 177.8)
- removed the P5 at (62.8, 177.8)
- removed the P5 at (218.8, 50.8)
- removed the P5 at (275.8, 50.8)
- removed the P5 at (275.8, 107.8)
- removed the P5 at (218.8, 107.8)
- removed the P5 at (62.8, 107.8)
- removed the P6 at (184.5, 177.8)
- removed the P6 at (85.5, 107.8)
- removed the P6 at (85.5, 50.8)
- removed the P6 at (241.5, 177.8)
- removed the P6 at (85.5, 177.8)
- removed the P6 at (28.5, 177.8)
- removed the P6 at (184.5, 50.8)
- removed the P6 at (241.5, 50.8)
- removed the P6 at (241.5, 107.8)
- removed the P6 at (184.5, 107.8)
- removed the P6 at (28.5, 107.8)
- removed the P7 at (184.5, 188.0)
- removed the P7 at (85.5, 118.0)
- removed the P7 at (85.5, 61.0)
- removed the P7 at (241.5, 188.0)
- removed the P7 at (85.5, 188.0)
- removed the P7 at (28.5, 188.0)
- removed the P7 at (184.5, 61.0)
- removed the P7 at (241.5, 61.0)
- removed the P7 at (241.5, 118.0)
- removed the P7 at (184.5, 118.0)
- removed the P7 at (28.5, 118.0)
- removed the Q1 at (203.5, 174.7)
- removed the Q1 at (104.5, 104.7)
- removed the Q1 at (104.5, 47.7)
- removed the Q1 at (260.5, 174.7)
- removed the Q1 at (104.5, 174.7)
- removed the Q1 at (47.5, 174.7)
- removed the Q1 at (203.5, 47.7)
- removed the Q1 at (260.5, 47.7)
- removed the Q1 at (260.5, 104.7)
- removed the Q1 at (203.5, 104.7)
- removed the Q1 at (47.5, 104.7)
- removed the R1 at (216.2, 162.0)
- removed the R1 at (117.2, 92.0)
- removed the R1 at (117.2, 35.0)
- removed the R1 at (273.2, 162.0)
- removed the R1 at (117.2, 162.0)
- removed the R1 at (60.2, 162.0)
- removed the R1 at (216.2, 35.0)
- removed the R1 at (273.2, 35.0)
- removed the R1 at (273.2, 92.0)
- removed the R1 at (216.2, 92.0)
- removed the R1 at (60.2, 92.0)
- removed the R2 at (213.0, 162.0)
- removed the R2 at (114.0, 92.0)
- removed the R2 at (114.0, 35.0)
- removed the R2 at (270.0, 162.0)
- removed the R2 at (114.0, 162.0)
- removed the R2 at (57.0, 162.0)
- removed the R2 at (213.0, 35.0)
- removed the R2 at (270.0, 35.0)
- removed the R2 at (270.0, 92.0)
- removed the R2 at (213.0, 92.0)
- removed the R2 at (57.0, 92.0)
- removed the R3 at (195.9, 161.3)
- removed the R3 at (96.9, 91.3)
- removed the R3 at (96.9, 34.3)
- removed the R3 at (252.9, 161.3)
- removed the R3 at (96.9, 161.3)
- removed the R3 at (39.9, 161.3)
- removed the R3 at (195.9, 34.3)
- removed the R3 at (252.9, 34.3)
- removed the R3 at (252.9, 91.3)
- removed the R3 at (195.9, 91.3)
- removed the R3 at (39.9, 91.3)
- removed the R4 at (204.8, 162.0)
- removed the R4 at (105.8, 92.0)
- removed the R4 at (105.8, 35.0)
- removed the R4 at (261.8, 162.0)
- removed the R4 at (105.8, 162.0)
- removed the R4 at (48.8, 162.0)
- removed the R4 at (204.8, 35.0)
- removed the R4 at (261.8, 35.0)
- removed the R4 at (261.8, 92.0)
- removed the R4 at (204.8, 92.0)
- removed the R4 at (48.8, 92.0)
- removed the R5 at (210.5, 179.7)
- removed the R5 at (111.5, 109.7)
- removed the R5 at (111.5, 52.7)
- removed the R5 at (267.5, 179.7)
- removed the R5 at (111.5, 179.7)
- removed the R5 at (54.5, 179.7)
- removed the R5 at (210.5, 52.7)
- removed the R5 at (267.5, 52.7)
- removed the R5 at (267.5, 109.7)
- removed the R5 at (210.5, 109.7)
- removed the R5 at (54.5, 109.7)
- removed the R6 at (213.0, 179.7)
- removed the R6 at (114.0, 109.7)
- removed the R6 at (114.0, 52.7)
- removed the R6 at (270.0, 179.7)
- removed the R6 at (114.0, 179.7)
- removed the R6 at (57.0, 179.7)
- removed the R6 at (213.0, 52.7)
- removed the R6 at (270.0, 52.7)
- removed the R6 at (270.0, 109.7)
- removed the R6 at (213.0, 109.7)
- removed the R6 at (57.0, 109.7)
- removed the R7 at (190.8, 165.1)
- removed the R7 at (91.8, 95.1)
- removed the R7 at (91.8, 38.1)
- removed the R7 at (247.8, 165.1)
- removed the R7 at (91.8, 165.1)
- removed the R7 at (34.8, 165.1)
- removed the R7 at (190.8, 38.1)
- removed the R7 at (247.8, 38.1)
- removed the R7 at (247.8, 95.1)
- removed the R7 at (190.8, 95.1)
- removed the R7 at (34.8, 95.1)
- removed the U1 at (204.1, 167.7)
- removed the U1 at (105.1, 97.7)
- removed the U1 at (105.1, 40.7)
- removed the U1 at (261.1, 167.7)
- removed the U1 at (105.1, 167.7)
- removed the U1 at (48.1, 167.7)
- removed the U1 at (204.1, 40.7)
- removed the U1 at (261.1, 40.7)
- removed the U1 at (261.1, 97.7)
- removed the U1 at (204.1, 97.7)
- removed the U1 at (48.1, 97.7)
- added C1: 10uF/25V, C1P_D2, F.Cu at (190.3, 42.0)
- added C1: 10uF/25V, C1P_D2, F.Cu at (76.3, 94.0)
- added C1: 10uF/25V, C1P_D2, F.Cu at (76.3, 42.0)
- added C1: 10uF/25V, C1P_D2, F.Cu at (242.3, 42.0)
- added C1: 10uF/25V, C1P_D2, F.Cu at (242.3, 94.0)
- added C1: 10uF/25V, C1P_D2, F.Cu at (190.3, 94.0)
- added C1: 10uF/25V, C1P_D2, F.Cu at (190.3, 173.9)
- added C1: 10uF/25V, C1P_D2, F.Cu at (242.3, 173.9)
- added C1: 10uF/25V, C1P_D2, F.Cu at (76.3, 173.9)
- added C1: 10uF/25V, C1P_D2, F.Cu at (24.3, 173.9)
- added C1: 10uF/25V, C1P_D2, F.Cu at (24.3, 94.0)
- added D1: LED, LED3, F.Cu at (218.9, 38.1)
- added D1: LED, LED3, F.Cu at (104.9, 90.1)
- added D1: LED, LED3, F.Cu at (104.9, 38.1)
- added D1: LED, LED3, F.Cu at (270.9, 38.1)
- added D1: LED, LED3, F.Cu at (270.9, 90.1)
- added D1: LED, LED3, F.Cu at (218.9, 90.1)
- added D1: LED, LED3, F.Cu at (218.9, 170.1)
- added D1: LED, LED3, F.Cu at (270.9, 170.1)
- added D1: LED, LED3, F.Cu at (104.9, 170.1)
- added D1: LED, LED3, F.Cu at (52.9, 170.1)
- added D1: LED, LED3, F.Cu at (52.9, 90.1)
- added D2: BZX55C15, D3, F.Cu at (185.3, 44.5)
- added D2: BZX55C15, D3, F.Cu at (71.3, 96.5)
- added D2: BZX55C15, D3, F.Cu at (71.3, 44.5)
- added D2: BZX55C15, D3, F.Cu at (237.3, 44.5)
- added D2: BZX55C15, D3, F.Cu at (237.3, 96.5)
- added D2: BZX55C15, D3, F.Cu at (185.3, 96.5)
- added D2: BZX55C15, D3, F.Cu at (185.3, 176.5)
- added D2: BZX55C15, D3, F.Cu at (237.3, 176.5)
- added D2: BZX55C15, D3, F.Cu at (71.3, 176.5)
- added D2: BZX55C15, D3, F.Cu at (19.3, 176.5)
- added D2: BZX55C15, D3, F.Cu at (19.3, 96.5)
- added DP5050: , DP5050, F.Cu at (205.0, 39.0)
- added DP5050: , DP5050, F.Cu at (91.0, 91.0)
- added DP5050: , DP5050, F.Cu at (91.0, 39.0)
- added DP5050: , DP5050, F.Cu at (39.0, 39.0)
- added DP5050: , DP5050, F.Cu at (257.0, 39.0)
- added DP5050: , DP5050, F.Cu at (257.0, 91.0)
- added DP5050: , DP5050, F.Cu at (205.0, 91.0)
- added DP5050: , DP5050, F.Cu at (205.0, 171.0)
- added DP5050: , DP5050, F.Cu at (257.0, 171.0)
- added DP5050: , DP5050, F.Cu at (91.0, 171.0)
- added DP5050: , DP5050, F.Cu at (39.0, 171.0)
- added DP5050: , DP5050, F.Cu at (39.0, 91.0)
- added F1: FUSE, AUTOFUSE, F.Cu at (203.0, 20.4)
- added F1: FUSE, AUTOFUSE, F.Cu at (89.0, 72.4)
- added F1: FUSE, AUTOFUSE, F.Cu at (89.0, 20.4)
- added F1: FUSE, AUTOFUSE, F.Cu at (255.0, 20.4)
- added F1: FUSE, AUTOFUSE, F.Cu at (255.0, 72.4)
- added F1: FUSE, AUTOFUSE, F.Cu at (203.0, 72.4)
- added F1: FUSE, AUTOFUSE, F.Cu at (203.0, 152.4)
- added F1: FUSE, AUTOFUSE, F.Cu at (255.0, 152.4)
- added F1: FUSE, AUTOFUSE, F.Cu at (89.0, 152.4)
- added F1: FUSE, AUTOFUSE, F.Cu at (37.0, 152.4)
- added F1: FUSE, AUTOFUSE, F.Cu at (37.0, 72.4)
- added P1: IN+, HEADER_6.3, F.Cu at (187.8, 28.0)
- added P1: IN+, HEADER_6.3, F.Cu at (73.8, 80.0)
- added P1: IN+, HEADER_6.3, F.Cu at (73.8, 28.0)
- added P1: IN+, HEADER_6.3, F.Cu at (239.8, 28.0)
- added P1: IN+, HEADER_6.3, F.Cu at (239.8, 80.0)
- added P1: IN+, HEADER_6.3, F.Cu at (187.8, 80.0)
- added P1: IN+, HEADER_6.3, F.Cu at (187.8, 160.0)
- added P1: IN+, HEADER_6.3, F.Cu at (239.8, 160.0)
- added P1: IN+, HEADER_6.3, F.Cu at (73.8, 160.0)
- added P1: IN+, HEADER_6.3, F.Cu at (21.8, 160.0)
- added P1: IN+, HEADER_6.3, F.Cu at (21.8, 80.0)
- added P2: IN-, HEADER_6.3, F.Cu at (187.8, 35.6)
- added P2: IN-, HEADER_6.3, F.Cu at (73.8, 87.6)
- added P2: IN-, HEADER_6.3, F.Cu at (73.8, 35.6)
- added P2: IN-, HEADER_6.3, F.Cu at (239.8, 35.6)
- added P2: IN-, HEADER_6.3, F.Cu at (239.8, 87.6)
- added P2: IN-, HEADER_6.3, F.Cu at (187.8, 87.6)
- added P2: IN-, HEADER_6.3, F.Cu at (187.8, 167.6)
- added P2: IN-, HEADER_6.3, F.Cu at (239.8, 167.6)
- added P2: IN-, HEADER_6.3, F.Cu at (73.8, 167.6)
- added P2: IN-, HEADER_6.3, F.Cu at (21.8, 167.6)
- added P2: IN-, HEADER_6.3, F.Cu at (21.8, 87.6)
- added P3: LED, HDR-2, F.Cu at (224.6, 40.7)
- added P3: LED, HDR-2, F.Cu at (110.6, 92.7)
- added P3: LED, HDR-2, F.Cu at (110.6, 40.7)
- added P3: LED, HDR-2, F.Cu at (276.6, 40.7)
- added P3: LED, HDR-2, F.Cu at (276.6, 92.7)
- added P3: LED, HDR-2, F.Cu at (224.6, 92.7)
- added P3: LED, HDR-2, F.Cu at (224.6, 172.7)
- added P3: LED, HDR-2, F.Cu at (276.6, 172.7)
- added P3: LED, HDR-2, F.Cu at (110.6, 172.7)
- added P3: LED, HDR-2, F.Cu at (58.6, 172.7)
- added P3: LED, HDR-2, F.Cu at (58.6, 92.7)
- added P4: SW_IN, HDR-2, F.Cu at (224.6, 50.8)
- added P4: SW_IN, HDR-2, F.Cu at (110.6, 102.8)
- added P4: SW_IN, HDR-2, F.Cu at (110.6, 50.8)
- added P4: SW_IN, HDR-2, F.Cu at (276.6, 50.8)
- added P4: SW_IN, HDR-2, F.Cu at (276.6, 102.8)
- added P4: SW_IN, HDR-2, F.Cu at (224.6, 102.8)
- added P4: SW_IN, HDR-2, F.Cu at (224.6, 182.8)
- added P4: SW_IN, HDR-2, F.Cu at (276.6, 182.8)
- added P4: SW_IN, HDR-2, F.Cu at (110.6, 182.8)
- added P4: SW_IN, HDR-2, F.Cu at (58.6, 182.8)
- added P4: SW_IN, HDR-2, F.Cu at (58.6, 102.8)
- added P5: SENSE, HDR-2, F.Cu at (224.6, 45.8)
- added P5: SENSE, HDR-2, F.Cu at (110.6, 97.8)
- added P5: SENSE, HDR-2, F.Cu at (110.6, 45.8)
- added P5: SENSE, HDR-2, F.Cu at (276.6, 45.8)
- added P5: SENSE, HDR-2, F.Cu at (276.6, 97.8)
- added P5: SENSE, HDR-2, F.Cu at (224.6, 97.8)
- added P5: SENSE, HDR-2, F.Cu at (224.6, 177.8)
- added P5: SENSE, HDR-2, F.Cu at (276.6, 177.8)
- added P5: SENSE, HDR-2, F.Cu at (110.6, 177.8)
- added P5: SENSE, HDR-2, F.Cu at (58.6, 177.8)
- added P5: SENSE, HDR-2, F.Cu at (58.6, 97.8)
- added P6: OUT+, HEADER_6.3, F.Cu at (192.2, 55.9)
- added P6: OUT+, HEADER_6.3, F.Cu at (78.2, 107.9)
- added P6: OUT+, HEADER_6.3, F.Cu at (78.2, 55.9)
- added P6: OUT+, HEADER_6.3, F.Cu at (244.2, 55.9)
- added P6: OUT+, HEADER_6.3, F.Cu at (244.2, 107.9)
- added P6: OUT+, HEADER_6.3, F.Cu at (192.2, 107.9)
- added P6: OUT+, HEADER_6.3, F.Cu at (192.2, 187.9)
- added P6: OUT+, HEADER_6.3, F.Cu at (244.2, 187.9)
- added P6: OUT+, HEADER_6.3, F.Cu at (78.2, 187.9)
- added P6: OUT+, HEADER_6.3, F.Cu at (26.2, 187.9)
- added P6: OUT+, HEADER_6.3, F.Cu at (26.2, 107.9)
- added P7: OUT-, HEADER_6.3, F.Cu at (201.1, 55.9)
- added P7: OUT-, HEADER_6.3, F.Cu at (87.1, 107.9)
- added P7: OUT-, HEADER_6.3, F.Cu at (87.1, 55.9)
- added P7: OUT-, HEADER_6.3, F.Cu at (253.1, 55.9)
- added P7: OUT-, HEADER_6.3, F.Cu at (253.1, 107.9)
- added P7: OUT-, HEADER_6.3, F.Cu at (201.1, 107.9)
- added P7: OUT-, HEADER_6.3, F.Cu at (201.1, 187.9)
- added P7: OUT-, HEADER_6.3, F.Cu at (253.1, 187.9)
- added P7: OUT-, HEADER_6.3, F.Cu at (87.1, 187.9)
- added P7: OUT-, HEADER_6.3, F.Cu at (35.1, 187.9)
- added P7: OUT-, HEADER_6.3, F.Cu at (35.1, 107.9)
- added Q1: IRFZ44VBF, TO220, F.Cu at (210.7, 43.2)
- added Q1: IRFZ44VBF, TO220, F.Cu at (96.7, 95.2)
- added Q1: IRFZ44VBF, TO220, F.Cu at (96.7, 43.2)
- added Q1: IRFZ44VBF, TO220, F.Cu at (262.7, 43.2)
- added Q1: IRFZ44VBF, TO220, F.Cu at (262.7, 95.2)
- added Q1: IRFZ44VBF, TO220, F.Cu at (210.7, 95.2)
- added Q1: IRFZ44VBF, TO220, F.Cu at (210.7, 175.2)
- added Q1: IRFZ44VBF, TO220, F.Cu at (262.7, 175.2)
- added Q1: IRFZ44VBF, TO220, F.Cu at (96.7, 175.2)
- added Q1: IRFZ44VBF, TO220, F.Cu at (44.7, 175.2)
- added Q1: IRFZ44VBF, TO220, F.Cu at (44.7, 95.2)
- added R1: 10K, R4, F.Cu at (221.5, 29.2)
- added R1: 10K, R4, F.Cu at (107.5, 81.2)
- added R1: 10K, R4, F.Cu at (107.5, 29.2)
- added R1: 10K, R4, F.Cu at (273.5, 29.2)
- added R1: 10K, R4, F.Cu at (273.5, 81.2)
- added R1: 10K, R4, F.Cu at (221.5, 81.2)
- added R1: 10K, R4, F.Cu at (221.5, 161.2)
- added R1: 10K, R4, F.Cu at (273.5, 161.2)
- added R1: 10K, R4, F.Cu at (107.5, 161.2)
- added R1: 10K, R4, F.Cu at (55.5, 161.2)
- added R1: 10K, R4, F.Cu at (55.5, 81.2)
- added R2: 10K, R4, F.Cu at (218.9, 29.2)
- added R2: 10K, R4, F.Cu at (104.9, 81.2)
- added R2: 10K, R4, F.Cu at (104.9, 29.2)
- added R2: 10K, R4, F.Cu at (270.9, 29.2)
- added R2: 10K, R4, F.Cu at (270.9, 81.2)
- added R2: 10K, R4, F.Cu at (218.9, 81.2)
- added R2: 10K, R4, F.Cu at (218.9, 161.2)
- added R2: 10K, R4, F.Cu at (270.9, 161.2)
- added R2: 10K, R4, F.Cu at (104.9, 161.2)
- added R2: 10K, R4, F.Cu at (52.9, 161.2)
- added R2: 10K, R4, F.Cu at (52.9, 81.2)
- added R3: R005/1W, R4_5_6, F.Cu at (199.2, 35.6)
- added R3: R005/1W, R4_5_6, F.Cu at (85.2, 87.6)
- added R3: R005/1W, R4_5_6, F.Cu at (85.2, 35.6)
- added R3: R005/1W, R4_5_6, F.Cu at (251.2, 35.6)
- added R3: R005/1W, R4_5_6, F.Cu at (251.2, 87.6)
- added R3: R005/1W, R4_5_6, F.Cu at (199.2, 87.6)
- added R3: R005/1W, R4_5_6, F.Cu at (199.2, 167.6)
- added R3: R005/1W, R4_5_6, F.Cu at (251.2, 167.6)
- added R3: R005/1W, R4_5_6, F.Cu at (85.2, 167.6)
- added R3: R005/1W, R4_5_6, F.Cu at (33.2, 167.6)
- added R3: R005/1W, R4_5_6, F.Cu at (33.2, 87.6)
- added R4: 100K, R4, F.Cu at (208.8, 32.4)
- added R4: 100K, R4, F.Cu at (94.8, 84.4)
- added R4: 100K, R4, F.Cu at (94.8, 32.4)
- added R4: 100K, R4, F.Cu at (260.8, 32.4)
- added R4: 100K, R4, F.Cu at (260.8, 84.4)
- added R4: 100K, R4, F.Cu at (208.8, 84.4)
- added R4: 100K, R4, F.Cu at (208.8, 164.4)
- added R4: 100K, R4, F.Cu at (260.8, 164.4)
- added R4: 100K, R4, F.Cu at (94.8, 164.4)
- added R4: 100K, R4, F.Cu at (42.8, 164.4)
- added R4: 100K, R4, F.Cu at (42.8, 84.4)
- added R5: 10R, R4, F.Cu at (218.3, 52.1)
- added R5: 10R, R4, F.Cu at (104.3, 104.1)
- added R5: 10R, R4, F.Cu at (104.3, 52.1)
- added R5: 10R, R4, F.Cu at (270.3, 52.1)
- added R5: 10R, R4, F.Cu at (270.3, 104.1)
- added R5: 10R, R4, F.Cu at (218.3, 104.1)
- added R5: 10R, R4, F.Cu at (218.3, 184.1)
- added R5: 10R, R4, F.Cu at (270.3, 184.1)
- added R5: 10R, R4, F.Cu at (104.3, 184.1)
- added R5: 10R, R4, F.Cu at (52.3, 184.1)
- added R5: 10R, R4, F.Cu at (52.3, 104.1)
- added R6: 100K, R4, F.Cu at (220.8, 52.1)
- added R6: 100K, R4, F.Cu at (106.8, 104.1)
- added R6: 100K, R4, F.Cu at (106.8, 52.1)
- added R6: 100K, R4, F.Cu at (272.8, 52.1)
- added R6: 100K, R4, F.Cu at (272.8, 104.1)
- added R6: 100K, R4, F.Cu at (220.8, 104.1)
- added R6: 100K, R4, F.Cu at (220.8, 184.1)
- added R6: 100K, R4, F.Cu at (272.8, 184.1)
- added R6: 100K, R4, F.Cu at (106.8, 184.1)
- added R6: 100K, R4, F.Cu at (54.8, 184.1)
- added R6: 100K, R4, F.Cu at (54.8, 104.1)
- added R7: 6K8 (48V), R4, F.Cu at (195.4, 35.6)
- added R7: 6K8 (48V), R4, F.Cu at (81.4, 87.6)
- added R7: 6K8 (48V), R4, F.Cu at (81.4, 35.6)
- added R7: 6K8 (48V), R4, F.Cu at (247.4, 35.6)
- added R7: 6K8 (48V), R4, F.Cu at (247.4, 87.6)
- added R7: 6K8 (48V), R4, F.Cu at (195.4, 87.6)
- added R7: 6K8 (48V), R4, F.Cu at (195.4, 167.6)
- added R7: 6K8 (48V), R4, F.Cu at (247.4, 167.6)
- added R7: 6K8 (48V), R4, F.Cu at (81.4, 167.6)
- added R7: 6K8 (48V), R4, F.Cu at (29.4, 167.6)
- added R7: 6K8 (48V), R4, F.Cu at (29.4, 87.6)
- added U1: INA168, SOT23-5, B.Cu at (208.8, 35.6)
- added U1: INA168, SOT23-5, B.Cu at (94.8, 87.6)
- added U1: INA168, SOT23-5, B.Cu at (94.8, 35.6)
- added U1: INA168, SOT23-5, B.Cu at (260.8, 35.6)
- added U1: INA168, SOT23-5, B.Cu at (260.8, 87.6)
- added U1: INA168, SOT23-5, B.Cu at (208.8, 87.6)
- added U1: INA168, SOT23-5, B.Cu at (208.8, 167.6)
- added U1: INA168, SOT23-5, B.Cu at (260.8, 167.6)
- added U1: INA168, SOT23-5, B.Cu at (94.8, 167.6)
- added U1: INA168, SOT23-5, B.Cu at (42.8, 167.6)
- added U1: INA168, SOT23-5, B.Cu at (42.8, 87.6)
- moved F1 9.54 mm to (37.0, 20.4)
- moved P7 8.39 mm to (35.1, 55.9), turned to 90 degrees
- moved P1 8.38 mm to (21.8, 28.0)
- moved R1 7.43 mm to (55.5, 29.2)
- moved U1 7.41 mm to (42.8, 35.6)
- moved C1 7.13 mm to (24.3, 42.0)
- moved D2 7.13 mm to (19.3, 44.5)
- moved P2 7.13 mm to (21.8, 35.6)
- moved R2 7.05 mm to (52.9, 29.2)
- moved D1 7.05 mm to (52.9, 38.1)
- moved R3 6.78 mm to (33.2, 35.6)
- moved P5 6.54 mm to (58.6, 45.8)
- moved P3 6.54 mm to (58.6, 40.7)
- moved P4 6.54 mm to (58.6, 50.8)
- moved R4 6.54 mm to (42.8, 32.4)
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Routing:
- net N-000006: track 2396.0 -> 1734.2 mm
- net N-000007: track 643.6 -> 473.3 mm
- net N-000004: track 383.8 -> 319.5 mm
- net N-0000011: track 731.2 -> 791.2 mm
- net N-000003: track 435.9 -> 486.4 mm
- net N-000008: track 385.5 -> 434.4 mm
- net N-000002: track 114.8 -> 160.6 mm
- net N-000001: track 53.3 -> 79.9 mm
- net N-000005: track 66.0 -> 76.7 mm
- net N-0000010: track 278.5 -> 282.7 mm
Other:
- outline, holes or cut-outs redrawn
